File: ChainReaction_CV_core.kicad_pcb (KiCad board)
At the start: 2 copper layers, 38.1 x 99.1 mm, 31 parts, among them J15 conn_L, J16 conn_R, J17 power_bus, U1 4017, U2 TL074, U3 4013

Commit message: Fixed problems: - added power-on reset function - added 100ks to discharge caps with FFs(4013) - only for the CV; adjusted the parameter (100k -> 10k) of a resistor with a FF
Parts:
- added C13: 1u, Capacitor_THT:CP_Radial_D5.0mm_P2.50mm, F.Cu at (81.3, 74.9)
- added D45: D, Diode_THT:D_DO-34_SOD68_P2.54mm_Vertical_AnodeUp, F.Cu at (82.5, 94.0)
- added D46: D, Diode_THT:D_DO-34_SOD68_P2.54mm_Vertical_AnodeUp, F.Cu at (81.3, 82.5)
- added D47: D, Diode_THT:D_DO-34_SOD68_P2.54mm_Vertical_AnodeUp, F.Cu at (109.2, 91.4)
- added R67: 100k, Resistor_THT:R_Axial_DIN0207_L6.3mm_D2.5mm_P2.54mm_Vertical, F.Cu at (81.3, 80.0)
- added R68: 100k, Resistor_THT:R_Axial_DIN0207_L6.3mm_D2.5mm_P2.54mm_Vertical, F.Cu at (78.7, 85.1)
- added R69: 100k, Resistor_THT:R_Axial_DIN0207_L6.3mm_D2.5mm_P2.54mm_Vertical, F.Cu at (104.1, 68.6)
- added R70: 100k, Resistor_THT:R_Axial_DIN0207_L6.3mm_D2.5mm_P2.54mm_Vertical, F.Cu at (106.7, 66.0)
- added R71: 10k, Resistor_THT:R_Axial_DIN0207_L6.3mm_D2.5mm_P7.62mm_Horizontal, F.Cu at (99.1, 83.8)
- added R72: 1M, Resistor_THT:R_Axial_DIN0207_L6.3mm_D2.5mm_P2.54mm_Vertical, F.Cu at (106.7, 76.2)
- added R73: 100k, Resistor_THT:R_Axial_DIN0207_L6.3mm_D2.5mm_P2.54mm_Vertical, F.Cu at (88.9, 104.1)
- R64: renamed from R63; value 100k -> 10k
- renumbered C13 to C14, C14 to C15, C15 to C16, D45 to D48, D46 to D49, R64 to R63
Connections:
- D43 pad 1: /CV_Logic/EoC_in -> /CV_Logic/Q8
- R60 pad 1: /CV_Logic/EoC_in -> /CV_Logic/Q8
- U1 pad 13: /CV_Logic/EoC_in -> /CV_Logic/Q8
- U1 pad 9: /CV_Logic/EoC_in -> /CV_Logic/Q8
- U2 pad 10: GND -> Net-(R71-Pad2)
- U2 pad 8: Net-(U2-Pad8) -> Net-(D47-Pad2)
- U2 pad 9: Net-(U2-Pad8) -> Net-(R69-Pad1)
Routing:
- net /CV_Logic/Q8: track 0.00 -> 58.7 mm
- net Net-(D45-Pad1): track 0.00 -> 30.3 mm
- net /CV_Logic/EoC_in: track 55.2 -> 30.5 mm
- net +12V: track 164.2 -> 187.3 mm
- net Net-(D47-Pad2): track 0.00 -> 19.9 mm
- net Net-(R71-Pad2): track 0.00 -> 17.3 mm
- net Net-(C13-Pad2): track 0.00 -> 7.64 mm
- net Net-(R69-Pad1): track 0.00 -> 6.13 mm
- net Net-(D44-Pad2): track 46.8 -> 50.8 mm
- net -12V: track 152.8 -> 156.0 mm
- net Net-(D42-Pad2): track 36.1 -> 38.8 mm
- net Net-(U2-Pad8): track 2.54 -> 0.00 mm
- net /CV_Logic/cv_out: track 43.8 -> 44.8 mm
- net /CV_Logic/Q3: track 37.0 -> 37.6 mm
Other:
- board text added: "ChainReaction CV ver. 1.1"
- board text removed: "ChainReaction CV ver. 1"
