File: ChainReaction_Gate_interface.kicad_pcb (KiCad board)
At the start: 2 copper layers, 38.1 x 99.1 mm, 110 parts, among them J10 conn_L, J11 clock_out, J12 EoC, J13 trigger_out, J14 conn_R, J8 clock, J9 reset, SW1 Gate1, SW2 Gate2, SW3 Gate3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

Commit message: Fixed problems: - added power-on reset function - added 100ks to discharge caps with FFs(4013) - only for the CV; adjusted the parameter (100k -> 10k) of a resistor with a FF
Routing:
- net Net-(C4-Pad2): track 15.2 -> 13.6 mm
