File: _module_trigger_logic.sch (KiCad schematic (older format))
At the start: 46 parts, among them J18 conn_L, J19 conn_R, J20 power_bus, U4 4017, U5 TL072, U6 4013, U7 TL074

Commit message: Fixed problems: - added power-on reset function - added 100ks to discharge caps with FFs(4013) - only for the CV; adjusted the parameter (100k -> 10k) of a resistor with a FF
Parts:
- added C20: 1u, Capacitor_THT:CP_Radial_D5.0mm_P2.50mm, symbol Device:CP
- added D54: D, Diode_THT:D_DO-34_SOD68_P2.54mm_Vertical_AnodeUp, symbol Device:D
- added R79: 10k, Resistor_THT:R_Axial_DIN0207_L6.3mm_D2.5mm_P2.54mm_Vertical, symbol Device:R
- added R83: 1M, Resistor_THT:R_Axial_DIN0207_L6.3mm_D2.5mm_P2.54mm_Vertical, symbol Device:R
- renumbered C16 to C17, C17 to C18, C18 to C19, C19 to C21, C20 to C22, C21 to C23, C22 to C24, C23 to C25, D47 to D50, D48 to D51, D49 to D52, D50 to D53, D51 to D55, D52 to D56, D53 to D57, D56 to D58, D54 to D59, D55 to D60, R67 to R74, R68 to R75, R69 to R76, R70 to R77, R71 to R78, R72 to R80, R73 to R81, R74 to R82, R80 to R84, R75 to R85, R76 to R86, R77 to R87, R81 to R88, R78 to R89, R79 to R90, R82 to R91, R83 to R92, R84 to R93, R85 to R94, R86 to R95, R87 to R96
Connections:
- net +12V: now also C20.1
- net EoC_in: now also R79.2
- net GND: now also R79.1, R83.1
- net stop: now also D54.1 (K)
- new net: C20.2, D54.2 (A), R83.2
Other:
- note added: "2022-09-05 10k on breadboard\n-> 2022-09-21 implemented with 100k"
- note added: "power-on reset"
- note added: "to discharge C18"
- note removed: "2022-09-05 10k on breadboard"
